File: Eagle/SCH.brd (EAGLE design)
At the start: 97.8 x 46.7 mm, 28 parts, among them IC1 L7805, IC2 L7805, Q1 IRF540, Q2 IRF540, Q3 IRF540

Commit message: Update PCB
Parts:
- moved C2 1.80 mm to (-19.1, 3.81)
- moved IC2 1.80 mm to (-17.8, -3.81)
- moved IC1 1.80 mm to (-17.8, -12.7)
- moved C1 1.42 mm to (-16.5, 8.26)
Routing:
- net N$4: track 37.1 -> 39.2 mm
- net GND: track 249.8 -> 251.4 mm
- net +5V: track 117.2 -> 118.0 mm
Changed lines of the file:
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@@
 <drawing>
 <settings>
-<setting alwaysvectorfont="yes"/>
+<setting alwaysvectorfont="no"/>
 <setting verticaltext="up"/>
 </settings>
@@
 <attribute name="VALUE" x="-38.1" y="15.875" size="1.27" layer="27" rot="R180"/>
 </element>
-<element name="C1" library="rcl" library_urn="urn:adsk.eagle:library:334" package="C025-024X044" package3d_urn="urn:adsk.eagle:package:23630/1" value="10uF" x="-17.78" y="7.62" smashed="yes" rot="R180">
-<attribute name="NAME" x="-15.494" y="8.255" size="1.27" layer="25" ratio="10" rot="R270"/>
-<attribute name="SPICEPREFIX" value="C" x="-17.78" y="7.62" size="1.778" layer="27" rot="R180" display="off"/>
-</element>
-<element name="C2" library="rcl" library_urn="urn:adsk.eagle:library:334" package="C025-024X044" package3d_urn="urn:adsk.eagle:package:23630/1" value="10uF" x="-20.32" y="2.54" smashed="yes">
-<attribute name="NAME" x="-24.13" y="1.778" size="1.27" layer="25" ratio="10" rot="R90"/>
-<attribute name="SPICEPREFIX" value="C" x="-20.32" y="2.54" size="1.778" layer="27" display="off"/>
-<attribute name="VALUE" x="-22.733" y="0.889" size="1.27" layer="27" ratio="10" rot="R90"/>
+<element name="C1" library="rcl" library_urn="urn:adsk.eagle:library:334" package="C025-024X044" package3d_urn="urn:adsk.eagle:package:23630/1" value="10uF" x="-16.51" y="8.255" smashed="yes" rot="R180">
+<attribute name="NAME" x="-14.224" y="8.89" size="1.27" layer="25" ratio="10" rot="R270"/>
+<attribute name="SPICEPREFIX" value="C" x="-16.51" y="8.255" size="1.778" layer="27" rot="R180" display="off"/>
+</element>
+<element name="C2" library="rcl" library_urn="urn:adsk.eagle:library:334" package="C025-024X044" package3d_urn="urn:adsk.eagle:package:23630/1" value="10uF" x="-19.05" y="3.81" smashed="yes">
+<attribute name="NAME" x="-22.86" y="3.048" size="1.27" layer="25" ratio="10" rot="R90"/>
+<attribute name="SPICEPREFIX" value="C" x="-19.05" y="3.81" size="1.778" layer="27" display="off"/>
+<attribute name="VALUE" x="-21.463" y="2.159" size="1.27" layer="27" ratio="10" rot="R90"/>
 </element>
 <element name="C3" library="capacitor-wima" library_urn="urn:adsk.eagle:library:116" package="C5B2.5" package3d_urn="urn:adsk.eagle:package:5426/1" value="470uF" x="35.56" y="-2.54" smashed="yes" rot="R180">
@@
 <attribute name="VALUE" x="-15.24" y="-29.845" size="1.27" layer="27"/>
 </element>
-<element name="IC1" library="linear" library_urn="urn:adsk.eagle:library:262" package="TO220V" package3d_urn="urn:adsk.eagle:package:16417/1" value="L7805" x="-19.05" y="-11.43" smashed="yes" rot="R180">
-<attribute name="NAME" x="-23.495" y="-5.6388" size="1.27" layer="25" ratio="10" rot="R180"/>
-<attribute name="VALUE" x="-12.319" y="-8.128" size="1.27" layer="27" ratio="10" rot="R90"/>
-</element>
-<element name="IC2" library="linear" library_urn="urn:adsk.eagle:library:262" package="TO220V" package3d_urn="urn:adsk.eagle:package:16417/1" value="L7805" x="-19.05" y="-5.08" smashed="yes" rot="R180">
-<attribute name="NAME" x="-15.621" y="-0.5842" size="1.27" layer="25" ratio="10"/>
+<element name="IC1" library="linear" library_urn="urn:adsk.eagle:library:262" package="TO220V" package3d_urn="urn:adsk.eagle:package:16417/1" value="L7805" x="-17.78" y="-12.7" smashed="yes" rot="R180">
+<attribute name="NAME" x="-22.225" y="-6.9088" size="1.27" layer="25" ratio="10" rot="R180"/>
+<attribute name="VALUE" x="-11.049" y="-9.398" size="1.27" layer="27" ratio="10" rot="R90"/>
+</element>
+<element name="IC2" library="linear" library_urn="urn:adsk.eagle:library:262" package="TO220V" package3d_urn="urn:adsk.eagle:package:16417/1" value="L7805" x="-17.78" y="-3.81" smashed="yes" rot="R180">
+<attribute name="NAME" x="-14.351" y="0.6858" size="1.27" layer="25" ratio="10"/>
 </element>
 <element name="JP1" library="pinhead" library_urn="urn:adsk.eagle:library:325" package="1X02" package3d_urn="urn:adsk.eagle:package:22435/2" value="" x="15.24" y="-15.24" smashed="yes">
@@
 <via x="3.302" y="-25.4" extent="1-16" drill="0.35"/>
 <wire x1="3.302" y1="-25.4" x2="6.858" y2="-25.4" width="1.27" layer="16"/>
-<wire x1="-19.05" y1="-8.89" x2="-19.05" y2="-2.54" width="1.27" layer="16"/>
-<wire x1="-19.05" y1="-2.54" x2="-19.05" y2="2.54" width="1.27" layer="16"/>
-<wire x1="-19.05" y1="2.54" x2="-19.05" y2="7.62" width="1.27" layer="16"/>
+<wire x1="-17.78" y1="-10.16" x2="-17.78" y2="-1.27" width="1.27" layer="16"/>
+<wire x1="-17.78" y1="-1.27" x2="-17.78" y2="3.81" width="1.27" layer="16"/>
+<wire x1="-17.78" y1="3.81" x2="-17.78" y2="8.255" width="1.27" layer="16"/>
 <wire x1="-19.304" y1="-15.621" x2="-31.976" y2="-15.621" width="1.27" layer="16"/>
-<wire x1="-19.304" y1="-15.621" x2="-19.05" y2="-15.367" width="1.27" layer="16"/>
-<wire x1="-19.05" y1="-15.367" x2="-19.05" y2="-8.89" width="1.27" layer="16"/>
+<wire x1="-17.907" y1="-15.621" x2="-17.78" y2="-15.494" width="1.27" layer="16"/>
+<wire x1="-17.78" y1="-15.494" x2="-17.78" y2="-10.16" width="1.27" layer="16"/>
 <wire x1="-3.81" y1="-12.7" x2="-10.16" y2="-12.7" width="1.27" layer="16"/>
-<wire x1="-19.304" y1="-15.621" x2="-13.335" y2="-15.621" width="1.27" layer="16"/>
-<wire x1="-25.4" y1="11.43" x2="-21.59" y2="7.62" width="1.27" layer="16"/>
-<wire x1="-21.59" y1="7.62" x2="-19.05" y2="7.62" width="1.27" layer="16"/>
+<wire x1="-17.907" y1="-15.621" x2="-13.335" y2="-15.621" width="1.27" layer="16"/>
+<wire x1="-25.4" y1="11.43" x2="-22.225" y2="8.255" width="1.27" layer="16"/>
+<wire x1="-22.225" y1="8.255" x2="-17.78" y2="8.255" width="1.27" layer="16"/>
 <wire x1="-1.27" y1="2.54" x2="-5.08" y2="2.54" width="1.27" layer="16"/>
 <wire x1="-5.08" y1="2.54" x2="-10.16" y2="-2.54" width="1.27" layer="16"/>
@@
 <wire x1="38.1" y1="-1.27" x2="38.1" y2="-2.54" width="1.27" layer="16"/>
 <wire x1="3.302" y1="-12.827" x2="3.302" y2="-25.4" width="1.27" layer="16"/>
+<wire x1="-19.304" y1="-15.621" x2="-17.907" y2="-15.621" width="1.27" layer="16"/>
 <polygon width="1.27" layer="16" spacing="2.54" isolate="1">
 <vertex x="-49.53" y="17.78"/>
@@
 <contactref element="IC1" pad="1"/>
 <contactref element="IC2" pad="1"/>
-<wire x1="-16.51" y1="-8.89" x2="-16.51" y2="-2.54" width="1.27" layer="16"/>
-<wire x1="-16.51" y1="-2.54" x2="-16.51" y2="7.62" width="1.27" layer="16"/>
+<wire x1="-15.24" y1="-10.16" x2="-15.24" y2="-1.27" width="1.27" layer="16"/>
+<wire x1="-15.24" y1="-1.27" x2="-15.24" y2="8.255" width="1.27" layer="16"/>
 <wire x1="-30.48" y1="-8.89" x2="-30.48" y2="-11.43" width="1.27" layer="1"/>
-<wire x1="-17.907" y1="-13.081" x2="-16.51" y2="-11.684" width="1.27" layer="1"/>
-<wire x1="-16.51" y1="-11.684" x2="-16.51" y2="-8.89" width="1.27" layer="1"/>
+<wire x1="-16.256" y1="-13.081" x2="-15.24" y2="-12.065" width="1.27" layer="1"/>
+<wire x1="-15.24" y1="-12.065" x2="-15.24" y2="-10.16" width="1.27" layer="1"/>
 <wire x1="-30.48" y1="-11.43" x2="-28.829" y2="-13.081" width="1.27" layer="1"/>
-<wire x1="-28.829" y1="-13.081" x2="-17.907" y2="-13.081" width="1.27" layer="1"/>
+<wire x1="-28.829" y1="-13.081" x2="-16.256" y2="-13.081" width="1.27" layer="1"/>
 </signal>
 <signal name="+5V">
@@
 <wire x1="-39.695" y1="-18.88" x2="-39.695" y2="-14.295" width="1.27" layer="16"/>
 <wire x1="-39.695" y1="-14.295" x2="-38.481" y2="-13.081" width="1.27" layer="16"/>
-<wire x1="-38.481" y1="-13.081" x2="-25.781" y2="-13.081" width="1.27" layer="16"/>
-<wire x1="-25.781" y1="-13.081" x2="-21.59" y2="-8.89" width="1.27" layer="16"/>
-<wire x1="-21.59" y1="2.54" x2="-21.59" y2="3.81" width="1.27" layer="1"/>
-<wire x1="-21.59" y1="3.81" x2="-20.32" y2="5.08" width="1.27" layer="1"/>
-<wire x1="-10.16" y1="5.08" x2="-2.54" y2="12.7" width="1.27" layer="1"/>
-<wire x1="-20.32" y1="5.08" x2="-10.16" y2="5.08" width="1.27" layer="1"/>
+<wire x1="-38.481" y1="-13.081" x2="-23.241" y2="-13.081" width="1.27" layer="16"/>
+<wire x1="-23.241" y1="-13.081" x2="-20.32" y2="-10.16" width="1.27" layer="16"/>
+<wire x1="-20.32" y1="3.81" x2="-18.161" y2="5.969" width="1.27" layer="1"/>
+<wire x1="-9.271" y1="5.969" x2="-2.54" y2="12.7" width="1.27" layer="1"/>
+<wire x1="-18.161" y1="5.969" x2="-9.271" y2="5.969" width="1.27" layer="1"/>
 <wire x1="15.24" y1="6.35" x2="15.24" y2="3.81" width="1.27" layer="1"/>
 <wire x1="15.24" y1="3.81" x2="16.51" y2="2.54" width="1.27" layer="1"/>
@@
 <wire x1="31.115" y1="-9.525" x2="30.48" y2="-10.16" width="0.6096" layer="1"/>
 <wire x1="30.48" y1="-10.16" x2="29.21" y2="-10.16" width="0.6096" layer="1"/>
-<wire x1="-21.59" y1="2.54" x2="-21.59" y2="-2.54" width="1.27" layer="1"/>
-<wire x1="-21.59" y1="-2.54" x2="-21.59" y2="-8.89" width="1.27" layer="1"/>
+<wire x1="-20.32" y1="3.81" x2="-20.32" y2="-1.27" width="1.27" layer="1"/>
+<wire x1="-20.32" y1="-1.27" x2="-20.32" y2="-10.16" width="1.27" layer="1"/>
 </signal>
 <signal name="D5">
@@
 <contactref element="Q3" pad="D"/>
 <contactref element="JP5" pad="2"/>
-<wire x1="-18.97" y1="15.24" x2="-18.97" y2="15.16" width="1.27" layer="16"/>
-<wire x1="-18.97" y1="15.16" x2="-8.89" y2="5.08" width="1.27" layer="16"/>
-<wire x1="-8.89" y1="5.08" x2="-1.27" y2="5.08" width="1.27" layer="16"/>
+<wire x1="-7.62" y1="5.08" x2="-1.27" y2="5.08" width="1.27" layer="16"/>
+<wire x1="-18.97" y1="15.24" x2="-15.16" y2="11.43" width="1.27" layer="16"/>
+<wire x1="-15.16" y1="11.43" x2="-13.97" y2="11.43" width="1.27" layer="16"/>
+<wire x1="-13.97" y1="11.43" x2="-7.62" y2="5.08" width="1.27" layer="16"/>
 </signal>
 <signal name="N$13">
